Commit message: premier bras robot

File: src/mon_bras/urdf/mon_bras.urdf (robot description, URDF)
Before this commit: robot mon_bras, 2 links, 1 joints
Links:
- added link lien2; visual cylinder length=0.15 radius=0.025
- added link lien3; visual cylinder length=0.12 radius=0.02
- added link lien4; visual cylinder length=0.1 radius=0.018
- added link lien5; visual cylinder length=0.08 radius=0.015
- added link lien6; visual box size=0.05 0.05 0.02
- link lien1: geometry visual cylinder length=0.15 radius=0.03
Joints:
- added joint joint2: type revolute, parent lien1, child lien2, origin xyz=0 0 0.15, axis 0 1 0, limit lower=-1.57 upper=1.57 effort=10 velocity=1
- added joint joint3: type revolute, parent lien2, child lien3, origin xyz=0 0 0.15, axis 0 1 0, limit lower=-1.57 upper=1.57 effort=10 velocity=1
- added joint joint4: type revolute, parent lien3, child lien4, origin xyz=0 0 0.12, axis 0 0 1, limit lower=-3.14 upper=3.14 effort=10 velocity=1
- added joint joint5: type revolute, parent lien4, child lien5, origin xyz=0 0 0.1, axis 0 1 0, limit lower=-1.57 upper=1.57 effort=10 velocity=1
- added joint joint6: type revolute, parent lien5, child lien6, origin xyz=0 0 0.08, axis 0 0 1, limit lower=-3.14 upper=3.14 effort=10 velocity=1
- joint joint1: axis (none) -> 0 0 1; limit (none) -> lower=-3.14 upper=3.14 effort=10 velocity=1; type fixed -> revolute

Commit message: ajout urdf avec collision

File: src/mon_bras/urdf/mon_bras.urdf (robot description, URDF)
Before this commit: robot mon_bras, 7 links, 6 joints
Links:
- link base: mass None -> 1.0; geometry collision box size=0.1 0.1 0.05; visual box size=0.1 0.1 0.05
- link lien1: mass None -> 0.5; geometry collision cylinder length=0.15 radius=0.03; visual cylinder length=0.15 radius=0.03
- link lien2: mass None -> 0.5; geometry collision cylinder length=0.15 radius=0.025; visual cylinder length=0.15 radius=0.025
- link lien3: mass None -> 0.3; geometry collision cylinder length=0.12 radius=0.02; visual cylinder length=0.12 radius=0.02
- link lien4: mass None -> 0.3; geometry collision cylinder length=0.1 radius=0.018; visual cylinder length=0.1 radius=0.018
- link lien5: mass None -> 0.2; geometry collision cylinder length=0.08 radius=0.015; visual cylinder length=0.08 radius=0.015
- link lien6: mass None -> 0.1; geometry collision box size=0.05 0.05 0.02; visual box size=0.05 0.05 0.02
